File: Hardware/OpenBook.brd (EAGLE design)
At the start: 175.6 x 111.8 mm, 103 parts, among them IC1 XC6220A331MR-G, IC5 BD5229G-TR, J1 FH34SRJ-24S-0.5SH_99_, J2 SAMACSYS_PARTS_USB4110-GF-A, J3 QWIIC_RIGHT_ANGLE, J4 112A-TAAR-R03_ATTEND, Q1 20V/4.2A/52mΩ/1.4W, Q2 20V/4.2A/52mΩ/1.4W, Q3 SI1308EDL-T1-GE3, U1 W25Q512JVEIQ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

Commit message: fixed issues.
Parts:
- moved J4 5.94 mm to (-4.91, 104.2)
- moved CHANGE_BUTTON 3.28 mm to (54.9, 117.0)
- moved C9 3.24 mm to (10.0, 96.5)
- moved C6 2.57 mm to (19.0, 116.9)
- moved BOOT_BUTTON 2.57 mm to (15.3, 117.1)
- moved RESET_BUTTON 1.69 mm to (39.4, 117.0)
- moved J2 0.82 mm to (159.1, 60.7)
- moved IC5 0.20 mm to (25.6, 109.2)
Routing:
- net GND: track 916.6 -> 934.0 mm
- net 3V3: track 465.5 -> 475.3 mm
- net MISO: track 261.6 -> 269.6 mm
- net IO/CHANGE: track 79.6 -> 86.2 mm
- net SS_SD: track 218.2 -> 212.2 mm
- net MOSI: track 235.6 -> 230.0 mm
- net N$15: track 23.5 -> 19.1 mm
- net RESET: track 132.4 -> 135.3 mm
- net EPD_DC: track 125.3 -> 123.9 mm
- net DP: track 22.3 -> 23.3 mm
- net SCK: track 265.3 -> 266.3 mm
- net VUSB: track 41.7 -> 42.7 mm
- net N$20: track 12.3 -> 13.1 mm
