File: Hardware/OpenBook.sch (EAGLE design)
At the start: 103 parts, among them IC1 XC6220A331MR-G, IC5 BD5229G-TR, J1 FH34SRJ-24S-0.5SH_99_, J2 SAMACSYS_PARTS_USB4110-GF-A, J3 QWIIC_RIGHT_ANGLE, J4 112A-TAAR-R03_ATTEND, Q1 20V/4.2A/52mΩ/1.4W, Q2 20V/4.2A/52mΩ/1.4W, Q3 SI1308EDL-T1-GE3, U1 W25Q512JVEIQ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

Commit message: fixed issues.
Other:
- note added: "Battery ChargeLevel"
- note added: "Display Type Selector"
- note added: "E-Paper Display Header"
- note added: "E-Paper Drive Circuit"
- note added: "EPD Power"
- note added: "ESP32 C6"
- note added: "Environmental Sensor BME688"
- note added: "External NORFlash64MB"
- note added: "LDO Voltage Regulator"
- note added: "Li-Po Battery Charging Controller"
- note added: "Qwiic / Stemma QT"
- note added: "RTC Module DS3231SN"
- note added: "SD Card"
- note added: "SPI ESD Protection Lines"
- note added: "Test Pads"
- note added: "USB C connector & ESD protection"
- note added: "Voltage Supervisor + Reset & Boot / IO Button"
- moved on the sheet: C1, C10_SUPERCAP, C1_BAT1, C1_BAT2, C2, C3, C8, D2, D7, EPD_C1, EPD_C10, EPD_C11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
